Commit message: Fixed error in Indigo.

File: youbot_description/urdf/youbot_arm/arm.transmission.xacro (robot description, xacro)
@@ -7,44 +7,54 @@
 	<!-- reduction ratio must not to be 0-->
 	<xacro:macro name="youbot_arm_transmission" params="name">
-		<transmission name="${name}_trans_1">
+    <transmission name="${name}_trans_1">
       <type>transmission_interface/SimpleTransmission</type>
-			<actuator name="${name}_motor_1">
-        <hardwareInterface>EffortJointInterface</hardwareInterface>
-        <mechanicalReduction>1</mechanicalReduction>
-      </actuator>
-			<joint name="${name}_joint_1"/>
-		</transmission>
-		<transmission name="${name}_trans_2">
+        <joint name="${name}_joint_1">
+          <hardwareInterface>EffortJointInterface</hardwareInterface>
+        </joint>
+        <actuator name="${name}_motor_1">
+          <hardwareInterface>EffortJointInterface</hardwareInterface>
+          <mechanicalReduction>1</mechanicalReduction>
+        </actuator>
+     </transmission>
+    <transmission name="${name}_trans_2">
       <type>transmission_interface/SimpleTransmission</type>
-			<actuator name="${name}_motor_2">
-        <hardwareInterface>EffortJointInterface</hardwareInterface>
-        <mechanicalReduction>1</mechanicalReduction>
-      </actuator>
-			<joint name="${name}_joint_2"/>
-		</transmission>
-		<transmission name="${name}_trans_3">
+        <joint name="${name}_joint_2">
+          <hardwareInterface>EffortJointInterface</hardwareInterface>
+        </joint>
+        <actuator name="${name}_motor_2">
+          <hardwareInterface>EffortJointInterface</hardwareInterface>
+          <mechanicalReduction>1</mechanicalReduction>
+        </actuator>
+     </transmission>
+    <transmission name="${name}_trans_3">
       <type>transmission_interface/SimpleTransmission</type>
-			<actuator name="${name}_motor_3">
-        <hardwareInterface>EffortJointInterface</hardwareInterface>
-        <mechanicalReduction>1</mechanicalReduction>
-      </actuator>
-			<joint name="${name}_joint_3"/>
-		</transmission>
-		<transmission name="${name}_trans_4">
+        <joint name="${name}_joint_3">
+          <hardwareInterface>EffortJointInterface</hardwareInterface>
+        </joint>
+        <actuator name="${name}_motor_3">
+          <hardwareInterface>EffortJointInterface</hardwareInterface>
+          <mechanicalReduction>1</mechanicalReduction>
+        </actuator>
+     </transmission>
+    <transmission name="${name}_trans_4">
       <type>transmission_interface/SimpleTransmission</type>
-			<actuator name="${name}_motor_4">
-        <hardwareInterface>EffortJointInterface</hardwareInterface>
-        <mechanicalReduction>1</mechanicalReduction>
-      </actuator>
-			<joint name="${name}_joint_4"/>
-		</transmission>
-		<transmission name="${name}_trans_5">
+        <joint name="${name}_joint_4">
+          <hardwareInterface>EffortJointInterface</hardwareInterface>
+        </joint>
+        <actuator name="${name}_motor_4">
+          <hardwareInterface>EffortJointInterface</hardwareInterface>
+          <mechanicalReduction>1</mechanicalReduction>
+        </actuator>
+     </transmission>
+    <transmission name="${name}_trans_5">
       <type>transmission_interface/SimpleTransmission</type>
-			<actuator name="${name}_motor_5">
-        <hardwareInterface>EffortJointInterface</hardwareInterface>
-        <mechanicalReduction>1</mechanicalReduction>
-      </actuator>
-			<joint name="${name}_joint_5"/>
-		</transmission>
+        <joint name="${name}_joint_5">
+          <hardwareInterface>EffortJointInterface</hardwareInterface>
+        </joint>
+        <actuator name="${name}_motor_5">
+          <hardwareInterface>EffortJointInterface</hardwareInterface>
+          <mechanicalReduction>1</mechanicalReduction>
+        </actuator>
+     </transmission>
 	</xacro:macro>
 </robot>

File: youbot_description/urdf/youbot_base/base.transmission.xacro (robot description, xacro)
@@ -9,71 +9,87 @@
 	<xacro:macro name="youbot_base_transmission">
 	<!-- front left wheel -->
-		<transmission name="wheel_trans_fl">
+    <transmission name="wheel_trans_fl">
       <type>transmission_interface/SimpleTransmission</type>
-			<actuator name="wheel_motor_fl">
-        <hardwareInterface>VelocityJointInterface</hardwareInterface>
-        <mechanicalReduction>${wheel_mechanical_reduction}</mechanicalReduction>
-      </actuator>
-			<joint name="wheel_joint_fl" />
-		</transmission>
-		<transmission name="caster_trans_fl">
+        <joint name="wheel_joint_fl">
+          <hardwareInterface>VelocityJointInterface</hardwareInterface>
+        </joint>
+        <actuator name="wheel_motor_fl">
+          <hardwareInterface>VelocityJointInterface</hardwareInterface>
+          <mechanicalReduction>${wheel_mechanical_reduction}</mechanicalReduction>
+        </actuator>
+     </transmission>
+    <transmission name="caster_trans_fl">
       <type>transmission_interface/SimpleTransmission</type>
-   	  <actuator name="caster_motor_fl">
-        <hardwareInterface>VelocityJointInterface</hardwareInterface>
-        <mechanicalReduction>${caster_mechanical_reduction}</mechanicalReduction>
-      </actuator>
-      <joint name="caster_joint_fl" />
-    </transmission>
+        <joint name="caster_joint_fl">
+          <hardwareInterface>VelocityJointInterface</hardwareInterface>
+        </joint>
+        <actuator name="caster_motor_fl">
+          <hardwareInterface>VelocityJointInterface</hardwareInterface>
+          <mechanicalReduction>${wheel_mechanical_reduction}</mechanicalReduction>
+        </actuator>
+     </transmission>
 	  <!-- front right wheel -->
-	  <transmission name="wheel_trans_fr">
+    <transmission name="wheel_trans_fr">
       <type>transmission_interface/SimpleTransmission</type>
-		  <actuator name="wheel_motor_fr">
-        <hardwareInterface>VelocityJointInterface</hardwareInterface>
-        <mechanicalReduction>${wheel_mechanical_reduction}</mechanicalReduction>
-      </actuator>
-		  <joint name="wheel_joint_fr" />
-	  </transmission>
-	  <transmission name="caster_trans_fr">
+        <joint name="wheel_joint_fr">
+          <hardwareInterface>VelocityJointInterface</hardwareInterface>
+        </joint>
+        <actuator name="wheel_motor_fr">
+          <hardwareInterface>VelocityJointInterface</hardwareInterface>
+          <mechanicalReduction>${wheel_mechanical_reduction}</mechanicalReduction>
+        </actuator>
+     </transmission>
+    <transmission name="caster_trans_fr">
       <type>transmission_interface/SimpleTransmission</type>
-      <actuator name="caster_motor_fr" >
-        <hardwareInterface>VelocityJointInterface</hardwareInterface>
-        <mechanicalReduction>${caster_mechanical_reduction}</mechanicalReduction>
-      </actuator>
-    	<joint name="caster_joint_fr" />
-    </transmission>
+        <joint name="caster_joint_fr">
+          <hardwareInterface>VelocityJointInterface</hardwareInterface>
+        </joint>
+        <actuator name="caster_motor_fr">
+          <hardwareInterface>VelocityJointInterface</hardwareInterface>
+          <mechanicalReduction>${wheel_mechanical_reduction}</mechanicalReduction>
+        </actuator>
+     </transmission>
 	  <!-- back left wheel -->
-	  <transmission name="wheel_trans_bl">
+    <transmission name="wheel_trans_bl">
       <type>transmission_interface/SimpleTransmission</type>
-	    <actuator name="wheel_motor_bl" >
-        <hardwareInterface>VelocityJointInterface</hardwareInterface>
-        <mechanicalReduction>${wheel_mechanical_reduction}</mechanicalReduction>
-      </actuator>
-	    <joint name="wheel_joint_bl" />
-	  </transmission>
-	  <transmission name="caster_trans_bl">
+        <joint name="wheel_joint_bl">
+          <hardwareInterface>VelocityJointInterface</hardwareInterface>
+        </joint>
+        <actuator name="wheel_motor_bl">
+          <hardwareInterface>VelocityJointInterface</hardwareInterface>
+          <mechanicalReduction>${wheel_mechanical_reduction}</mechanicalReduction>
+        </actuator>
+     </transmission>
+    <transmission name="caster_trans_bl">
       <type>transmission_interface/SimpleTransmission</type>
-      <actuator name="caster_motor_bl" >
-        <hardwareInterface>VelocityJointInterface</hardwareInterface>
-        <mechanicalReduction>${caster_mechanical_reduction}</mechanicalReduction>
-      </actuator>
-    	<joint name="caster_joint_bl" />
-    </transmission>
+        <joint name="caster_joint_bl">
+          <hardwareInterface>VelocityJointInterface</hardwareInterface>
+        </joint>
+        <actuator name="caster_motor_bl">
+          <hardwareInterface>VelocityJointInterface</hardwareInterface>
+          <mechanicalReduction>${wheel_mechanical_reduction}</mechanicalReduction>
+        </actuator>
+     </transmission>
 	  <!-- back right wheel -->
-	  <transmission name="wheel_trans_br">
+    <transmission name="wheel_trans_br">
       <type>transmission_interface/SimpleTransmission</type>
-	    <actuator name="wheel_motor_br" >
-        <hardwareInterface>VelocityJointInterface</hardwareInterface>
-        <mechanicalReduction>${wheel_mechanical_reduction}</mechanicalReduction>
-      </actuator>
-		  <joint name="wheel_joint_br" />
-	  </transmission>
-	  <transmission name="caster_trans_br">
+        <joint name="wheel_joint_br">
+          <hardwareInterface>VelocityJointInterface</hardwareInterface>
+        </joint>
+        <actuator name="wheel_motor_br">
+          <hardwareInterface>VelocityJointInterface</hardwareInterface>
+          <mechanicalReduction>${wheel_mechanical_reduction}</mechanicalReduction>
+        </actuator>
+     </transmission>
+    <transmission name="caster_trans_br">
       <type>transmission_interface/SimpleTransmission</type>
-      <actuator name="caster_motor_br" >
-        <hardwareInterface>VelocityJointInterface</hardwareInterface>
-        <mechanicalReduction>${caster_mechanical_reduction}</mechanicalReduction>
-      </actuator>
-    	<joint name="caster_joint_br" />
-    </transmission>
+        <joint name="caster_joint_br">
+          <hardwareInterface>VelocityJointInterface</hardwareInterface>
+        </joint>
+        <actuator name="caster_motor_br">
+          <hardwareInterface>VelocityJointInterface</hardwareInterface>
+          <mechanicalReduction>${wheel_mechanical_reduction}</mechanicalReduction>
+        </actuator>
+     </transmission>
   </xacro:macro>
 </robot>

File: youbot_description/urdf/youbot_gripper/gripper.transmission.xacro (robot description, xacro)
@@ -4,21 +4,25 @@
        xmlns:interface="http://playerstage.sourceforge.net/gazebo/xmlschema/#interface"
        xmlns:xacro="http://ros.org/wiki/xacro">
-	<xacro:macro name="youbot_gripper_transmission" params="name">
-		<transmission name="${name}_finger_l_trans">
+    <xacro:macro name="youbot_gripper_transmission" params="name">
+    <transmission name="${name}_finger_l_trans">
       <type>transmission_interface/SimpleTransmission</type>
-			<actuator name="${name}_finger_l_motor">
-        <hardwareInterface>EffortJointInterface</hardwareInterface>
-        <mechanicalReduction>1</mechanicalReduction>
-      </actuator>
-			<joint name="${name}_finger_joint_l"/>
-		</transmission>
-		<transmission name="${name}_finger_r_trans">
+        <joint name="${name}_finger_joint_l">
+          <hardwareInterface>EffortJointInterface</hardwareInterface>
+        </joint>
+        <actuator name="${name}_finger_l_motor">
+          <hardwareInterface>EffortJointInterface</hardwareInterface>
+          <mechanicalReduction>1</mechanicalReduction>
+        </actuator>
+     </transmission>
+    <transmission name="${name}_finger_r_trans">
       <type>transmission_interface/SimpleTransmission</type>
-			<actuator name="${name}_finger_r_motor">
-        <hardwareInterface>EffortJointInterface</hardwareInterface>
-        <mechanicalReduction>1</mechanicalReduction>
-      </actuator>
-			<joint name="${name}_finger_joint_r"/>
-		</transmission>
-	</xacro:macro>
+        <joint name="${name}_finger_joint_r">
+          <hardwareInterface>EffortJointInterface</hardwareInterface>
+        </joint>
+        <actuator name="${name}_finger_r_motor">
+          <hardwareInterface>EffortJointInterface</hardwareInterface>
+          <mechanicalReduction>1</mechanicalReduction>
+        </actuator>
+     </transmission>
+    </xacro:macro>
 </robot>
